File: STM32WB Game Controller.kicad_pcb (KiCad board)
At the start: 4 copper layers, 71 x 29 mm, 65 parts, among them J1 USB_C_Receptacle_USB2.0_14P, J2 Conn_01x04_Pin, J3 Conn_Coaxial, J4 TC2030, J5 Conn_01x04_Pin, J6 Conn_01x04_Pin, SW1 SW_Push, U1 SPX3819M5-L-3-3, U2 STM32WB55CEU6, U3 LIS2HH12, X1 32MHz

Commit message: Cleaned up schematic and redid vias on pcb
Parts:
- D2: value LED -> Green
- FLT1: footprint LP Filter Footprint:DLF162500LT-5028A1 -> Additional:DLF162500LT-5028A1
- moved C1 4.94 mm to (111.5, 88.5), turned to -90 degrees
- moved D1 4.25 mm to (111.0, 98.5)
- moved C24 4.15 mm to (124.6, 102.2), turned to -90 degrees
- moved J4 3.57 mm to (119.0, 96.7)
- moved C16 3.05 mm to (119.8, 101.5)
- moved C23 2.37 mm to (126.4, 103.2), turned to -90 degrees
- moved C8 1.88 mm to (151.2, 92.5)
- moved R14 1.58 mm to (133.4, 102.0)
- moved C22 1.55 mm to (128.6, 104.5), turned to -90 degrees
- moved R7 1.31 mm to (110.5, 108.7)
- moved J1 1.27 mm to (117.0, 109.8)
- moved R6 1.27 mm to (123.3, 108.6)
- moved C18 1.25 mm to (152.8, 95.8)
- moved U3 1.10 mm to (128.4, 97.8)
- moved R1 1.08 mm to (114.4, 86.8), turned to 0 degrees
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- renumbered R10-11 to R10
Connections:
- C2 pad 1: Net-(U1-EN) -> +5V
- C3 pad 1: Net-(U1-EN) -> +5V
- R1 pad 2: Net-(U1-EN) -> +5V
- U1 pad 1: Net-(U1-EN) -> +5V
- U1 pad 3: Net-(U1-EN) -> +5V
Routing:
- net +5V: track 34.0 -> 56.5 mm
- net Net-(U1-EN): track 13.1 -> 0.00 mm
- net /USB_D+: track 38.2 -> 45.9 mm
- net /USB_D-: track 42.1 -> 49.5 mm
- net /SWD_CLK: track 18.1 -> 21.7 mm
- net /I2C_SLC: track 22.8 -> 26.3 mm
- net /SWD_DIO: track 19.4 -> 22.6 mm
- net /I2C_SDA: track 27.6 -> 30.7 mm
- net /SWD_TRC: track 21.0 -> 23.9 mm
- net /SWD_NRST: track 45.2 -> 47.8 mm
- net /I2C_INT1: track 9.42 -> 11.1 mm, vias 0 -> 2
- net /HSE_IN: track 5.88 -> 4.48 mm
- net Net-(J1-CC1): track 7.31 -> 8.15 mm
- net /HSE_OUT: track 4.90 -> 4.06 mm
- net GND: track 19.1 -> 18.3 mm, vias 160 -> 99
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- added copper zone on In1.Cu, net +3.3V
- removed copper zone on In1.Cu, net GND
