File: STM32WB Game Controller.kicad_sch (KiCad schematic)
At the start: 41 parts, among them J1 Conn_01x04_Pin, J2 Conn_Coaxial, J3 USB_C_Receptacle_USB2.0_14P, J4 TC2030, SW1 SW_Push, U1 MIC5365-3.3YD5, U2 STM32WB55CEUx, X1 32kHz768, X2 32MHz

Commit message: Finished layout and routing
Parts:
- removed C17, C18: 10p, Capacitor_SMD:C_0603_1608Metric, symbol Device:C
- removed D1: LED, LED_SMD:LED_0603_1608Metric, symbol Device:LED
- removed U1: MIC5365-3.3YD5, Package_TO_SOT_SMD:TSOT-23-5, symbol Regulator_Linear:MIC5365-3.3YD5
- removed X1: 32kHz768, Crystal:Crystal_SMD_2012-2Pin_2.0x1.2mm, symbol Device:Crystal
- added C20, C21, C23, C24, C4: 100n, Capacitor_SMD:C_0603_1608Metric, symbol Device:C
- added C22, C3, C5: 4u7, Capacitor_SMD:C_0805_2012Metric, symbol Device:C
- added D2: LED, LED_SMD:LED_0603_1608Metric, symbol Device:LED
- added FID1, FID2, FID3: Fiducial, Fiducial:Fiducial_1mm_Mask2mm, symbol Mechanical:Fiducial
- added H1, H2, H3, H4: MountingHole_Pad, MountingHole:MountingHole_2.2mm_M2_Pad, symbol Mechanical:MountingHole_Pad
- added J2, J6: Conn_01x04_Pin, Connector_Molex:Molex_PicoBlade_53048-0410_1x04_P1.25mm_Horizontal, symbol Connector:Conn_01x04_Pin
- added R1: 0R, Resistor_SMD:R_0603_1608Metric, symbol Device:R
- added R10, R11, R14, R15: 5k1, Resistor_SMD:R_0603_1608Metric, symbol Device:R
- added R16, R2, R4, R5: 220R, Resistor_SMD:R_0603_1608Metric, symbol Device:R
- added U1: SPX3819M5-L-3-3, Package_TO_SOT_SMD:SOT-23-5, symbol Regulator_Linear:SPX3819M5-L-3-3
- added U3: LIS2HH12, Package_LGA:LGA-12_2x2mm_P0.5mm, symbol Sensor_Motion:LIS2HH12
- C1, C2: value 4.7u -> 100n; footprint Capacitor_SMD:C_0805_2012Metric -> Capacitor_SMD:C_0603_1608Metric; Distributor Link https://www.mouser.com/ProductDetail/Samsung-Electro-Mechan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 -> https://www.mouser.com/ProductDetail/YAGEO/CC0603JRX7R9BB10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; Manufacturer Samsung Electro-Mechanics -> YAGEO; Manufacturer Part Number CL21A475KPFNNNE -> CC0603JRX7R9BB104
- C17: renamed from C14; value 4.7u -> 4u7
- C6: renamed from C3; value 4.7u -> 4u7
- C9: renamed from C6; value 4.7u -> 4u7
- U2: value STM32WB55CEUx -> STM32WB55CEU6
- renumbered C7 to C10, C8 to C11, C9 to C12, C10 to C13, C11 to C14, C12 to C15, C13 to C16, C15 to C18, C16 to C19, C19 to C25, C4 to C7, C5 to C8, D2 to D1, J3 to J1, J2 to J3, J1 to J5, R1 to R12, R2 to R13, R4 to R6, R5 to R7, R7 to R8, R6 to R9, X2 to X1
Connections:
- net +3.3V: now also C22.1, C23.1, C24.1, C5.1, J6.2 (Pin_2), R14.1, R15.1, U1.5 (OUT), U3.10 (Vdd_IO), U3.2 (~{CS}), U3.9 (Vdd); no longer C2.1, J5.1 (Pin_1)
- net +5V: now also R1.1
- net GND: now also C20.2, C21.2, C22.2, C23.2, C24.2, C3.2, C4.2, C5.2, H1.1, H2.1, H3.1, H4.1, J6.1 (Pin_1), R16.2, U1.2 (GND), U3.3 (SA0/SDO), U3.5 (RES), U3.6 (GND), U3.7 (GND), U3.8 (GND); no longer J5.4 (Pin_4), R3.1
- net LED_A: now also U2.5 (PB8), D2.2 (A); no longer U2.16 (PA7)
- net LED_C: now also D2.1 (K), R16.1; no longer R3.2
- net UART_RXC: now also J5.4 (Pin_4); no longer J5.3 (Pin_3)
- net UART_TXC: now also J5.3 (Pin_3); no longer J5.2 (Pin_2)
- net USB_D+: now also D1.3 (I/O2), J1.A6 (D+), J1.B6 (D+)
- net USB_D-: now also D1.1 (I/O1), J1.A7 (D-), J1.B7 (D-)
- net ADC_IN6: now reaches U2.10 (PA1)
- net ADC_IN6: now also C20.1, R11.2
- net GPIOA_4: now reaches U2.13 (PA4)
- net GPIOA_4: now also R2.2
- net GPIOA_5: now reaches U2.14 (PA5)
- net GPIOA_5: now also R3.2
- net GPIOA_6: now reaches U2.15 (PA6)
- net GPIOA_6: now also R4.2
- net I2C_INT2: now reaches U2.44 (PB4)
- net I2C_INT2: now also U3.11 (INT2)
- net I2C_INT1: now reaches U2.45 (PB5)
- net I2C_INT1: now also U3.12 (INT1)
- net I2C_SLC: now reaches U2.46 (PB6)
- net I2C_SLC: now also J6.3 (Pin_3), R14.2, U3.1 (SCL/SPC)
- net I2C_SDA: now reaches U2.47 (PB7)
- net I2C_SDA: now also J6.4 (Pin_4), R15.2, U3.4 (SDA/SDI)
- net ADC_IN5: now reaches U2.9 (PA0)
- net ADC_IN5: now also C21.1, R10.2
- net LSE_IN: no longer names the net of U2.2 (PC14)
- net LSE_OUT: no longer names the net of U2.3 (PC15)
- new net: C4.1, U1.4 (BP)
- new net: C2.1, C3.1, R1.2, U1.1 (IN), U1.3 (EN)
- new net ADC_IN5C: J5.1 (Pin_1), R10.1
- new net ADC_IN6C: J5.2 (Pin_2), R11.1
- new net GPIOA_4C: J2.1 (Pin_1), R2.1
- new net GPIOA_5C: J2.2 (Pin_2), R3.1
- new net GPIOA_6C: J2.3 (Pin_3), R4.1
- new net GPIOA_7: R5.2, U2.16 (PA7)
- new net GPIOA_7C: J2.4 (Pin_4), R5.1
- no-connect marks 19 -> 11
Other:
- note added: "ADC/UART Header"
- note added: "Accelerometer"
- note added: "Fiducial Markers"
- note added: "GPIOA Header"
- note added: "I2C Header"
- note added: "Mounting Holes"
- note removed: "(3.3-18)/220~=7mA"
- note removed: "UART Header"
- moved on the sheet: C18, C19, C25, D1, FLT1, J3, J4, J5, L3, R12, R13, R8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

Commit message: Cleaned up schematic and redid vias on pcb
Parts:
- D2: value LED -> Green
- FLT1: footprint LP Filter Footprint:DLF162500LT-5028A1 -> Additional:DLF162500LT-5028A1
Connections:
- net +5V: now also C2.1, C3.1, R1.2, U1.1 (Vin), U1.3 (EN)
Other:
- note added: "+5V to +3V3 LDO Regulator"
- note removed: "+5V to +3V LDO Regulator"
- moved on the sheet: C1, C2, C20, C21, C22, C23, C24, C3, C4, C5, D1, J1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
